File: green_uv_led_pcb/green_uv_led_pcb.kicad_sch (KiCad schematic)
At the start: 20 parts, among them J1 Conn_01x02_Socket, J2 Conn_01x02_Socket, J3 Conn_01x02_Socket, J4 Conn_01x02_Socket

Commit message: new board version
Parts:
- removed D12, D16, D4, D8: LED, LED_SMD:LED_PLCC-2_3.4x3.0mm_KA, symbol Device:LED
- added H1, H2, H3, H4: MountingHole, MountingHole:MountingHole_3.2mm_M3, symbol Mechanical:MountingHole
- D13, D14, D15, D5, D6, D7: footprint LED_SMD:LED_PLCC-2_3.4x3.0mm_KA -> LED_SMD:LED_Cree-XP
- J1: value Conn_01x02_Socket -> Green bank 1
- J2: value Conn_01x02_Socket -> UV bank 1
- J3: value Conn_01x02_Socket -> Green bank 2
- J4: value Conn_01x02_Socket -> UV bank 2
Connections:
- net at J1.2 (Pin_2): now also D3.1 (K)
- net at J2.2 (Pin_2): now also D7.1 (K)
- net at D15.1 (K): now also J4.2 (Pin_2)
- net at D11.1 (K): now also J3.2 (Pin_2)
Other:
- moved on the sheet: D10, D11, D13, D14, D15, D5, D6, D7, D9, J2, J3, J4
