File: pcbs/led_driver/led_driver.kicad_sch (KiCad schematic)
At the start: 21 parts, among them J1 Barrel_Jack, J2 greenLED, J3 Conn_Coaxial, J4 Conn_Coaxial, J5 UVLED, U1 RCD-24, U2 LM350_TO220_9V_output, U3 RCD-24

Commit message: update led der
Parts:
- removed A1: Arduino_Mega2560_R3_Shield, PCM_arduino-library:Arduino_Mega2560_R3_Shield, symbol PCM_arduino-library:Arduino_Mega2560_R3_Shield
- removed C5: 1uF, Capacitor_THT:CP_Radial_D4.0mm_P2.00mm, symbol Device:C_Polarized
- removed J1: Barrel_Jack, Connector_BarrelJack:BarrelJack_GCT_DCJ200-10-A_Horizontal, symbol Connector:Barrel_Jack
- removed J3, J4: Conn_Coaxial, Connector_JST:JST_XH_B2B-XH-A_1x02_P2.50mm_Vertical, symbol Connector:Conn_Coaxial
- removed U2: LM350_TO220_9V_output, Package_TO_SOT_THT:TO-220-3_Vertical, symbol Regulator_Linear:LM350_TO220
- added C5, C8: 1uF, Capacitor_THT:CP_Radial_Tantal_D4.5mm_P2.50mm, symbol Device:C
- added C7: C, Capacitor_THT:CP_Radial_Tantal_D4.5mm_P2.50mm, symbol Device:C
- added H1, H2, H3, H4: MountingHole, MountingHole:MountingHole_3.2mm_M3, symbol Mechanical:MountingHole
- added J1, J3, J4, J8: Conn_01x03_Pin, Connector_JST:JST_XH_B3B-XH-A_1x03_P2.50mm_Vertical, symbol Connector:Conn_01x03_Pin
- added J6: power_in, Connector_JST:JST_XH_B2B-XH-A_1x02_P2.50mm_Vertical, symbol Connector:Conn_01x02_Pin
- added J7, J9: UVLED, Connector_JST:JST_XH_B2B-XH-A_1x02_P2.50mm_Vertical, symbol Connector:Conn_01x02_Pin
- added L3, L4: 22uH, Inductor_THT:L_Radial_D6.0mm_P4.00mm, symbol Device:L
- added U2, U4: RCD-24, Converter_DCDC:Converter_DCDC_RECOM_RCD-24_THT, symbol Driver_LED:RCD-24
- C3: value 0.1uF -> C
- R1: value 10k -> R
- R3: value 1.5k -> R
Connections:
- net GND: now also C3.2, C5.1, C7.2, C8.1, J1.3 (Pin_3), J3.3 (Pin_3), J4.3 (Pin_3), J6.2 (Pin_2), J8.3 (Pin_3), U2.4 (GND), U4.4 (GND); no longer C3.1, R1.1
- net VCC: now also C5.2, C8.2, J6.1 (Pin_1), L3.1, L4.1; no longer C3.2
- net at R3.2: now also C7.1, U4.2 (Analogue_Dimming)
- net at R3.1: now also J8.2 (Pin_2); no longer R1.2
- net PWM1: no longer names the net of U1.3 (PWM/ON/OFF)
- net PWM1: now also J3.1 (Pin_1)
- net PWM2: no longer names the net of U3.3 (PWM/ON/OFF)
- net PWM2: now also J4.1 (Pin_1)
- net analogue1: no longer names the net of R2.1
- net analogue1: now also J3.2 (Pin_2)
- net analogue2: no longer names the net of R4.1
- net analogue2: now also J4.2 (Pin_2)
- new net: J9.1 (Pin_1), U4.5 (-Vout)
- new net: J9.2 (Pin_2), U4.6 (+Vout)
- new net: C3.1, R1.2, U2.2 (Analogue_Dimming)
- new net: L4.2, U4.1 (+Vin)
- new net: J1.2 (Pin_2), R1.1
- new net: J7.1 (Pin_1), U2.5 (-Vout)
- new net: J7.2 (Pin_2), U2.6 (+Vout)
- new net: J8.1 (Pin_1), U4.3 (PWM/ON/OFF)
- new net: J1.1 (Pin_1), U2.3 (PWM/ON/OFF)
- new net: L3.2, U2.1 (+Vin)
- no-connect marks 71 -> 0
