File: Hardware/PCB/custom_driver/custom_driver.kicad_pcb (KiCad board)
At the start: 2 copper layers, 90 x 60 mm, 23 parts, among them J1 Conn_01x02_Shielded, J2 Conn_01x02, J3 Conn_01x02_Shielded, J4 Conn_01x02_Shielded, J5 Conn_01x03_Shielded, J6 Conn_01x02_Shielded, J7 Conn_01x03_Shielded, J8 Conn_01x02_Shielded, J9 Conn_01x02, Q1 IRFZ44NPBF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

Commit message: upgraded the circuit and the gerber files
Parts:
- added R5: 1k, Resistor_THT:R_Axial_DIN0207_L6.3mm_D2.5mm_P7.62mm_Horizontal, F.Cu at (117.0, 109.0)
- added R6: 1k, Resistor_THT:R_Axial_DIN0207_L6.3mm_D2.5mm_P7.62mm_Horizontal, F.Cu at (109.0, 80.0)
- added R7: 1k, Resistor_THT:R_Axial_DIN0207_L6.3mm_D2.5mm_P7.62mm_Horizontal, F.Cu at (113.8, 97.0)
- added R8: 1k, Resistor_THT:R_Axial_DIN0207_L6.3mm_D2.5mm_P7.62mm_Horizontal, F.Cu at (113.0, 67.0)
- R1, R2, R3, R4: value R -> 6.8R
- moved Q1 3.00 mm to (122.0, 116.1)
- moved Q2 2.89 mm to (121.0, 85.1)
Routing:
- net +12V: track 165.3 -> 190.0 mm
- net D1: track 14.3 -> 23.4 mm
- net G2: track 31.9 -> 25.2 mm
- net D4: track 17.5 -> 23.8 mm
- net S2: track 27.3 -> 21.2 mm
- net S1: track 29.9 -> 25.2 mm
- net D3: track 16.0 -> 20.6 mm
- net G1: track 35.8 -> 32.6 mm
- net D2: track 15.6 -> 18.4 mm
- net GRO: track 54.8 -> 53.2 mm
- net S4: track 32.9 -> 32.3 mm
- net G3: track 30.5 -> 30.0 mm
- net S3: track 34.6 -> 34.1 mm
