File: Hardware/PCB/custom_driver/custom_driver.kicad_sch (KiCad schematic)
At the start: 19 parts, among them J1 Conn_01x02_Shielded, J2 Conn_01x02, J3 Conn_01x02_Shielded, J4 Conn_01x02_Shielded, J5 Conn_01x03_Shielded, J6 Conn_01x02_Shielded, J7 Conn_01x03_Shielded, J8 Conn_01x02_Shielded, J9 Conn_01x02, Q1 IRFZ44NPBF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

Commit message: upgraded the circuit and the gerber files
Parts:
- added H1, H2, H3, H4: MountingHole, MountingHole:MountingHole_3.2mm_M3, symbol Mechanical:MountingHole
- added R5, R6, R7, R8: 1k, Resistor_THT:R_Axial_DIN0207_L6.3mm_D2.5mm_P7.62mm_Horizontal, symbol Device:R
- R1, R2, R3, R4: value R -> 6.8R
Connections:
- net +12V: now also R5.2, R6.1, R7.2, R8.2
- net D1: now also R5.1
- net D2: now also R6.2
- net D3: now also R7.1
- net D4: now also R8.1
Other:
- moved on the sheet: J1, J8, Q1, Q2, R1, R2
